Commit message: move robot config to drivetrain.urdf.xacro

File: urdf/drivetrain.urdf.xacro (robot description, xacro)
@@ -9,4 +9,7 @@
     <xacro:include filename="$(find kinco_diff_controller)/urdf/robot_control.urdf.xacro" />
     <xacro:robot prefix="$(arg prefix)" />
-    <xacro:robot_control name="Kinco Differential Robot" prefix="$(arg prefix)" use_mock_hardware="$(arg use_mock_hardware)"/>
+    <xacro:robot_control
+        name="Kinco Differential Robot" prefix="$(arg prefix)"
+        port="/dev/ttyS0" left_id="1" right_id="2"
+        use_mock_hardware="$(arg use_mock_hardware)"/>
 </robot>

File: urdf/robot_control.urdf.xacro (robot description, xacro)
@@ -1,12 +1,12 @@
 <?xml version="1.0"?>
 <robot xmlns:xacro="http://www.ros.org/wiki/xacro">
-    <xacro:macro name="robot_control" params="name prefix use_mock_hardware">
+    <xacro:macro name="robot_control" params="name prefix use_mock_hardware port left_id right_id">
         <ros2_control name="${name}" type="system">
             <xacro:unless value="${use_mock_hardware}">
                 <hardware>
                     <plugin>kinco_diff_controller/DrivetrainSystemHardware</plugin>
-                    <param name="port">/dev/ttyUSB0</param>
-                    <param name="left_id">1</param>
-                    <param name="right_id">2</param>
+                    <param name="port">${port}</param>
+                    <param name="left_id">${left_id}</param>
+                    <param name="right_id">${right_id}</param>
                     <param name="max_speed">3000</param>
                     <param name="reverse">1</param>

Commit message: add actual URDF model of IOP robot

File: urdf/drivetrain.urdf.xacro (robot description, xacro)
@@ -4,6 +4,4 @@
     <xacro:arg name="use_mock_hardware" default="false" />
     <xacro:include filename="$(find kinco_diff_controller)/urdf/robot_description.urdf.xacro" />
-    <!-- Import Rviz colors -->
-    <xacro:include filename="$(find kinco_diff_controller)/urdf/robot_materials.urdf.xacro" />
     <!-- Import ros2_control description -->
     <xacro:include filename="$(find kinco_diff_controller)/urdf/robot_control.urdf.xacro" />

File: urdf/robot_description.urdf.xacro (robot description, xacro)
@@ -2,162 +2,333 @@
 <robot xmlns:xacro="http://www.ros.org/wiki/xacro">
     <xacro:macro name="robot" params="prefix">
-        <!-- Constants for robot dimensions -->
-        <xacro:property name="PI" value="3.1415926535897931"/>
-        <xacro:property name="base_mass" value="0.3" /> <!-- arbitrary value for base mass -->
-        <xacro:property name="base_width" value="0.1" />
-        <xacro:property name="base_length" value="0.1" />
-        <xacro:property name="base_height" value="0.05" />
-        <xacro:property name="wheel_mass" value="0.3" /> <!-- arbitrary value for wheel mass -->
-        <xacro:property name="wheel_len" value="0.020" />
-        <xacro:property name="wheel_radius" value="0.015" />
-        <xacro:property name="caster_wheel_mass" value="0.1" /> <!-- arbitrary value for caster wheel mass -->
-        <xacro:property name="caster_wheel_radius" value="0.015" />
-        <xacro:property name="z_offset" value="-${base_height/2}" /> <!-- Space btw top of beam and the each joint -->
-        <!-- Base Link -->
         <link name="${prefix}base_link">
-            <collision>
-                <origin xyz="0 0 0" rpy="0 0 0"/>
-                <geometry>
-                    <box size="${base_width} ${base_length} ${base_height}"/>
-                </geometry>
-            </collision>
-            <visual>
-                <origin xyz="0 0 ${base_height/2}" rpy="0 0 0"/>
-                <geometry>
-                    <box size="${base_width} ${base_length} ${base_height}"/>
-                </geometry>
-                <material name="orange"/>
-            </visual>
-            <inertial>
-                <origin xyz="0 0 0" rpy="0 0 0"/>
-                <mass value="${base_mass}"/>
-                <inertia
-                    ixx="${base_mass / 12.0 * (base_length*base_length + base_height*base_height)}" ixy="0.0" ixz="0.0"
-                    iyy="${base_mass / 12.0 * (base_height*base_height + base_width*base_width)}" iyz="0.0"
-                    izz="${base_mass / 12.0 * (base_width*base_width + base_length*base_length)}"/>
-            </inertial>
+            <inertial>
+                <origin xyz="0.00116919992599684 2.964698431418E-06 0.158519577597417" rpy="0 0 0" />
+                <mass value="78.0827274144149" />
+                <inertia ixx="2.50667109850897" ixy="0.0167986143339606" ixz="-0.00462248899685703" iyy="4.2145346225938" iyz="0.000106887843698203" izz="6.28232013006863" />
+            </inertial>
+            <visual>
+                <origin xyz="0 0 0" rpy="0 0 0" />
+                <geometry>
+                    <mesh filename="package://kinco_diff_controller/meshes/base.STL" />
+                </geometry>
+                <material name="">
+                    <color rgba="0.650980392156863 0.619607843137255 0.588235294117647 1" />
+                </material>
+            </visual>
+            <collision>
+                <origin xyz="0 0 0" rpy="0 0 0" />
+                <geometry>
+                    <mesh filename="package://kinco_diff_controller/meshes/base.STL" />
+                </geometry>
+            </collision>
+        </link>
+        <!-- <joint name="${prefix}base_joint" type="fixed">
+        <parent link="${prefix}base_footprint" />
+        <child link="${prefix}base_link" />
+        <origin xyz="0 0 0" rpy="0 0 0"/>
+        </joint> -->
+        <link name="${prefix}lchinh1">
+            <inertial>
+                <origin xyz="6.3527E-07 6.4052E-06 8.8161E-06" rpy="0 0 0" />
+                <mass value="0.3265" />
+                <inertia ixx="0.00067921" ixy="2.1629E-18" ixz="1.2457E-17" iyy="0.00038694" iyz="3.8673E-10" izz="0.00038694" />
+            </inertial>
+            <visual>
+                <origin xyz="0 0 0" rpy="0 0 0" />
+                <geometry>
+                    <mesh filename="package://kinco_diff_controller/meshes/lchinh1.STL" />
+                </geometry>
+                <material name="">
+                    <color rgba="0.50196 0.50196 0.50196 1" />
+                </material>
+            </visual>
+            <collision>
+                <origin xyz="0 0 0" rpy="0 0 0" />
+                <geometry>
+                    <mesh filename="package://kinco_diff_controller/meshes/lchinh1.STL" />
+                </geometry>
+            </collision>
         </link>
         <joint name="${prefix}left_wheel_joint" type="continuous">
+            <origin xyz="0 0.21908 0.062877" rpy="1.5708 0.0030806 1.5708" />
+            <parent link="${prefix}base_link" />
+            <child link="${prefix}lchinh1" />
+            <axis xyz="1 0 0" />
+        </joint>
+        <link name="${prefix}lchinh2">
+            <inertial>
+                <origin xyz="6.3527E-07 4.0168E-06 1.013E-05" rpy="0 0 0" />
+                <mass value="0.3265" />
+                <inertia ixx="0.00067921" ixy="7.1118E-18" ixz="9.5532E-18" iyy="0.00038694" iyz="2.7867E-10" izz="0.00038694" />
+            </inertial>
+            <visual>
+                <origin xyz="0 0 0" rpy="0 0 0" />
+                <geometry>
+                    <mesh filename="package://kinco_diff_controller/meshes/lchinh2.STL" />
+                </geometry>
+                <material name="">
+                    <color rgba="0.50196 0.50196 0.50196 1" />
+                </material>
+            </visual>
+            <collision>
+                <origin xyz="0 0 0" rpy="0 0 0" />
+                <geometry>
+                    <mesh filename="package://kinco_diff_controller/meshes/lchinh2.STL" />
+                </geometry>
+            </collision>
+        </link>
+        <joint name="${prefix}right_wheel_joint" type="continuous">
+            <origin xyz="0 -0.21908 0.062877" rpy="2.0284 -0.0030806 1.5708" />
+            <parent link="${prefix}base_link" />
+            <child link="${prefix}lchinh2" />
+            <axis xyz="0.99998 -0.0055274 0.0027218" />
+        </joint>
+        <link name="${prefix}lbphu1">
+            <inertial>
+                <origin xyz="0.00946264375129513 -0.0176723960529895 -0.00608687345053327" rpy="0 0 0" />
+                <mass value="0.0812397412253748" />
+                <inertia ixx="7.05605896099002E-05" ixy="4.67952096548945E-07" ixz="-6.32104020706617E-06" iyy="0.000101227602264477" iyz="-3.01006512726596E-07" izz="6.47999500417815E-05" />
+            </inertial>
+            <visual>
+                <origin xyz="0 0 0" rpy="0 0 0" />
+                <geometry>
+                    <mesh filename="package://kinco_diff_controller/meshes/lbphu1.STL" />
+                </geometry>
+                <material name="">
+                    <color rgba="0.686274509803922 0.658823529411765 0.63921568627451 1" />
+                </material>
+            </visual>
+            <collision>
+                <origin xyz="0 0 0" rpy="0 0 0" />
+                <geometry>
+                    <mesh filename="package://kinco_diff_controller/meshes/lbphu1.STL" />
+                </geometry>
+            </collision>
+        </link>
+        <joint name="${prefix}jbphu1" type="fixed">
+            <origin xyz="0.31938 0.18313 0.0747" rpy="1.5708 0 1.5708" />
+            <parent link="${prefix}base_link" />
+            <child link="${prefix}lbphu1" />
+            <axis xyz="0 -1 0" />
+        </joint>
+        <link name="${prefix}lphu1">
+            <inertial>
+                <origin xyz="0.0119989443232924 1.70501568419468E-09 -1.61823893174429E-09" rpy="0 0 0" />
+                <mass value="0.0588561914547071" />
+                <inertia ixx="2.10634561244654E-05" ixy="2.9837515375904E-14" ixz="1.48354974680888E-14" iyy="1.38903083736938E-05" iyz="-1.50091507401853E-12" izz="1.38903088244573E-05" />
+            </inertial>
+            <visual>
+                <origin xyz="0 0 0" rpy="0 0 0" />
+                <geometry>
+                    <mesh filename="package://kinco_diff_controller/meshes/lphu1.STL" />
+                </geometry>
+                <material name="">
+                    <color rgba="1 1 1 1" />
+                </material>
+            </visual>
+            <collision>
+                <origin xyz="0 0 0" rpy="0 0 0" />
+                <geometry>
+                    <mesh filename="package://kinco_diff_controller/meshes/lphu1.STL" />
+                </geometry>
+            </collision>
+        </link>
+        <joint name="${prefix}jphu1" type="fixed">
+            <origin xyz="-0.024995 -0.049695 0.0018095" rpy="0 -0.99918 0" />
+            <parent link="${prefix}lbphu1" />
+            <child link="${prefix}lphu1" />
+            <axis xyz="-1 0 0" />
+        </joint>
+        <link name="${prefix}lbphu2">
+            <inertial>
+                <origin xyz="-0.0112512989675595 0.03267239615527 4.39991287848329E-09" rpy="0 0 0" />
+                <mass value="0.0812397511313111" />
+                <inertia ixx="7.46266281902283E-05" ixy="5.56405620269323E-07" ixz="1.05535643802289E-11" iyy="0.00010122761651701" iyz="-6.77914973369374E-12" izz="6.0733928293755E-05" />
+            </inertial>
+            <visual>
+                <origin xyz="0 0 0" rpy="0 0 0" />
+                <geometry>
+                    <mesh filename="package://kinco_diff_controller/meshes/lbphu2.STL" />
+                </geometry>
+                <material name="">
+                    <color rgba="0.686274509803922 0.658823529411765 0.63921568627451 1" />
+                </material>
+            </visual>
+            <collision>
+                <origin xyz="0 0 0" rpy="0 0 0" />
+                <geometry>
+                    <mesh filename="package://kinco_diff_controller/meshes/lbphu2.STL" />
+                </geometry>
+            </collision>
+        </link>
+        <joint name="${prefix}jbphu2" type="fixed">
+            <origin xyz="0.31938 -0.18288 0.0897" rpy="-1.5708 0 -0.57871" />
+            <parent link="${prefix}base_link" />
+            <child link="${prefix}lbphu2" />
+            <axis xyz="0 1 0" />
+        </joint>
+        <link name="${prefix}lphu2">
+            <inertial>
+                <origin xyz="-0.0120010556766208 1.70501079921337E-09 -1.62239932599562E-09" rpy="0 0 0" />
+                <mass value="0.0588561914546423" />
+                <inertia ixx="2.1063456124443E-05" ixy="2.98257335018538E-14" ixz="1.55663695875061E-14" iyy="1.38903083736981E-05" iyz="-1.50091476570755E-12" izz="1.38903088244611E-05" />
+            </inertial>
+            <visual>
+                <origin xyz="0 0 0" rpy="0 0 0" />
+                <geometry>
+                    <mesh filename="package://kinco_diff_controller/meshes/lphu2.STL" />
+                </geometry>
+                <material name="">
+                    <color rgba="1 1 1 1" />
+                </material>
+            </visual>
+            <collision>
+                <origin xyz="0 0 0" rpy="0 0 0" />
+                <geometry>
+                    <mesh filename="package://kinco_diff_controller/meshes/lphu2.STL" />
+                </geometry>
+            </collision>
+        </link>
+        <joint name="${prefix}jphu2" type="fixed">
+            <origin xyz="0.022 0.064695 0.012" rpy="0 -1.5708 0" />
+            <parent link="${prefix}lbphu2" />
+            <child link="${prefix}lphu2" />
+            <axis xyz="-1 0 0" />
+        </joint>
+        <link name="${prefix}lbphu3">
+            <inertial>
+                <origin xyz="-0.0112512987405764 0.0326723959483828 3.88080700908233E-09" rpy="0 0 0" />
+                <mass value="0.0812397536824839" />
+                <inertia ixx="7.46266289376794E-05" ixy="5.56405684377692E-07" ixz="1.21728790969442E-11" iyy="0.000101227619883743" iyz="-6.77973950305887E-12" izz="6.07339310000421E-05" />
+            </inertial>
+            <visual>
+                <origin xyz="0 0 0" rpy="0 0 0" />
+                <geometry>
+                    <mesh filename="package://kinco_diff_controller/meshes/lbphu3.STL" />
+                </geometry>
+                <material name="">
+                    <color rgba="0.686274509803922 0.658823529411765 0.63921568627451 1" />
+                </material>
+            </visual>
+            <collision>
+                <origin xyz="0 0 0" rpy="0 0 0" />
+                <geometry>
+                    <mesh filename="package://kinco_diff_controller/meshes/lbphu3.STL" />
+                </geometry>
+            </collision>
+        </link>
+        <joint name="${prefix}jbphu3" type="fixed">
+            <origin xyz="-0.31863 0.18313 0.0897" rpy="-1.5708 0 3.1416" />
+            <parent link="${prefix}base_link" />
+            <child link="${prefix}lbphu3" />
+            <axis xyz="0 1 0" />
+        </joint>
+        <link name="${prefix}lphu3">
+            <inertial>
+                <origin xyz="0.0119999999999998 -2.21784146603454E-10 -3.31598748459783E-10" rpy="0 0 0" />
+                <mass value="0.0588561914567127" />
+                <inertia ixx="2.10634561252174E-05" ixy="1.35878504384566E-14" ixz="-9.08799413589546E-15" iyy="1.38903090958169E-05" iyz="-1.20252769127507E-12" izz="1.38903081021528E-05" />
+            </inertial>
+            <visual>
+                <origin xyz="0 0 0" rpy="0 0 0" />
+                <geometry>
+                    <mesh filename="package://kinco_diff_controller/meshes/lphu3.STL" />
+                </geometry>
+                <material name="">
+                    <color rgba="0.250980392156863 0.250980392156863 0.250980392156863 1" />
+                </material>
+            </visual>
+            <collision>
+                <origin xyz="0 0 0" rpy="0 0 0" />
+                <geometry>
+                    <mesh filename="package://kinco_diff_controller/meshes/lphu3.STL" />
+                </geometry>
+            </collision>
+        </link>
+        <joint name="${prefix}jphu3" type="fixed">
+            <origin xyz="0.022 0.064695 -0.012" rpy="1.9626 -1.5708 0" />
+            <parent link="${prefix}lbphu3" />
+            <child link="${prefix}lphu3" />
+            <axis xyz="-1 0 0" />
+        </joint>
+        <link name="${prefix}lbphu4">
+            <inertial>
+                <origin xyz="-0.00013615031454986 -0.017672396198252 -0.0112504775096143" rpy="0 0 0" />
+                <mass value="0.0812397612278049" />
+                <inertia ixx="6.07359732393891E-05" ixy="-6.72855516700748E-09" ixz="1.6810978297091E-07" iyy="0.000101227631072605" iyz="-5.56367639975508E-07" izz="7.46246003421395E-05" />
+            </inertial>
+            <visual>
+                <origin xyz="0 0 0" rpy="0 0 0" />
+                <geometry>
+                    <mesh filename="package://kinco_diff_controller/meshes/lbphu4.STL" />
+                </geometry>
+                <material name="">
+                    <color rgba="0.792156862745098 0.819607843137255 0.933333333333333 1" />
+                </material>
+            </visual>
+            <collision>
+                <origin xyz="0 0 0" rpy="0 0 0" />
+                <geometry>
+                    <mesh filename="package://kinco_diff_controller/meshes/lbphu4.STL" />
+                </geometry>
+            </collision>
+        </link>
+        <joint name="${prefix}jbphu4" type="fixed">
+            <origin xyz="-0.31863 -0.18288 0.0747" rpy="1.5708 0 1.5708" />
+            <parent link="${prefix}base_link" />
+            <child link="${prefix}lbphu4" />
+            <axis xyz="0 -1 0" />
+        </joint>
+        <link name="${prefix}lphu4">
+            <inertial>
+                <origin xyz="-0.0120010556442718 3.15797032968135E-09 -1.62441360362919E-09" rpy="0 0 0" />
+                <mass value="0.0588561914225415" />
+                <inertia ixx="2.1063456114227E-05" ixy="-2.253105819105E-13" ixz="1.10871181094577E-14" iyy="1.38903083735561E-05" iyz="-1.50168295974446E-12" izz="1.38903088255762E-05" />
+            </inertial>
+            <visual>
+                <origin xyz="0 0 0" rpy="0 0 0" />
+                <geometry>
+                    <mesh filename="package://kinco_diff_controller/meshes/lphu4.STL" />
+                </geometry>
+                <material name="">
+                    <color rgba="0.250980392156863 0.250980392156863 0.250980392156863 1" />
+                </material>
+            </visual>
+            <collision>
+                <origin xyz="0 0 0" rpy="0 0 0" />
+                <geometry>
+                    <mesh filename="package://kinco_diff_controller/meshes/lphu4.STL" />
+                </geometry>
+            </collision>
+        </link>
+        <joint name="${prefix}jphu4" type="fixed">
+            <origin xyz="0.012265 -0.049695 0.021853" rpy="1.5708 0.012101 0" />
+            <parent link="${prefix}lbphu4" />
+            <child link="${prefix}lphu4" />
+            <axis xyz="-1 0 0" />
+        </joint>
+        <link name="${prefix}lidar_link">
+            <visual>
+                <origin xyz="0.0 0.0 0.0" rpy="1.5707 0 4.71" />
+                <geometry>
+                    <mesh filename="package://kinco_diff_controller/meshes/rplidar.dae" scale="0.001 0.001 0.001"/>
+                </geometry>
+                <material name="LightGrey">
+                    <color rgba="0.7 0.7 0.7 1.0"/>
+                </material>
+            </visual>
+            <collision>
+                <origin xyz="0.0 0.0 0.0" rpy="1.5707 0 4.71" />
+                <geometry>
+                    <mesh filename="package://kinco_diff_controller/meshes/rplidar.dae" scale="0.001 0.001 0.001"/>
+                </geometry>
+            </collision>
+        </link>
+        <joint name="${prefix}lidar_joint" type="fixed">
             <parent link="${prefix}base_link"/>
-            <child link="${prefix}left_wheel"/>
-            <origin xyz="0 -${base_width/2} ${z_offset}" rpy="0 0 0"/>
-            <axis xyz="0 1 0"/>
-            <dynamics damping="0.2"/>
-            <limit effort="100" velocity="1.0"/>
-        </joint>
-        <!-- left wheel Link -->
-        <link name="${prefix}left_wheel">
-            <collision>
-                <origin xyz="0 0 0" rpy="${PI/2} 0 0"/>
-                <geometry>
-                    <cylinder length="${wheel_len}" radius="${wheel_radius}"/>
-                </geometry>
-            </collision>
-            <visual>
-                <origin xyz="0 0 0" rpy="${PI/2} 0 0"/>
-                <geometry>
-                    <cylinder length="${wheel_len}" radius="${wheel_radius}"/>
-                </geometry>
-                <material name="black"/>
-            </visual>
-            <inertial>
-                <origin xyz="0 0 0" rpy="${PI/2} 0 0"/>
-                <mass value="${wheel_mass}"/>
-                <inertia
-                    ixx="${wheel_mass / 12.0 * (3*wheel_radius*wheel_radius + wheel_len*wheel_len)}" ixy="0.0" ixz="0.0"
-                    iyy="${wheel_mass / 12.0 * (3*wheel_radius*wheel_radius + wheel_len*wheel_len)}" iyz="0.0"
-                    izz="${wheel_mass / 2.0 * wheel_radius*wheel_radius}"/>
-            </inertial>
-        </link>
-        <joint name="${prefix}right_wheel_joint" type="continuous">
-            <parent link="${prefix}base_link"/>
-            <child link="${prefix}right_wheel"/>
-            <origin xyz="0 ${base_width/2} ${z_offset}" rpy="0 0 0"/>
-            <axis xyz="0 1 0"/>
-            <dynamics damping="0.2"/>
-            <limit effort="100" velocity="1.0"/>
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